File: Electronic/pcb/atlas_haptic_pcb/atlas_haptic_pcb/schematics.brd (EAGLE design)
At the start: 160 x 100 mm, 35 parts, among them U1 ISO1541, U3 MCP4725, U4 LM833N

Commit message: Figure of the circuit is updated. Mechanical part is revised.
Parts:
- removed U$11, U$5: OPA549, OPA:1X05_LONGPADS
- added J5, J6, J7, J9, SNUBBER: Jumper, SparkFun-Connectors:1X02_LONGPADS
- added MOTOR_TERMINAL: (no value), SparkFun-Connectors:SCREWTERMINAL-5MM-2
- added R13: 0R1, SparkFun-Resistors:1206
- added R14: 1R0, SparkFun-Resistors:1206
- added U11, U5: OPA549, OPA:1X05_LONGPADS
- C12: value 0.01uF -> 1n
- J3: device SparkFun-Connectors:SCREWTERMINAL-5MM-2 -> SparkFun-Connectors:1X03_LONGPADS
- R11: value 0R1 -> 0R01
- U1: device OPA:ISO1541 -> OPA:DIP254P762X508-8
- moved D2 114.4 mm to (61.0, 76.2), turned to 270 degrees
- moved C2 111.0 mm to (61.1, 19.1), turned to 180 degrees
- moved C3 109.2 mm to (55.9, 27.9), turned to 270 degrees
- moved C1 107.0 mm to (61.0, 15.2), turned to 180 degrees
- moved C11 105.4 mm to (54.6, 53.3), turned to 90 degrees
- moved C10 104.2 mm to (58.4, 53.3), turned to 90 degrees
- moved J1 102.1 mm to (59.0, 6.67)
- moved J3 98.4 mm to (74.9, 12.7), turned to 90 degrees
- moved R12 97.7 mm to (55.9, 95.2)
- moved D1 97.1 mm to (53.3, 76.2), turned to 270 degrees
- moved C9 95.8 mm to (54.6, 61.0), turned to 270 degrees
- moved U2 95.6 mm to (67.3, 55.9), turned to 270 degrees
- moved C8 94.5 mm to (58.4, 61.0), turned to 270 degrees
- moved R4 92.7 mm to (45.8, 11.5), turned to 90 degrees
- moved R7 91.4 mm to (39.4, 40.6), turned to 180 degrees
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Connections:
- removed net 3.3V: C12.2, R11.1
- removed net N$8: J3.2, R11.2, U$11.2
- new net N$11: J7.1, J9.1, R14.2
- new net N$12: J5.2, J6.2, J7.2, J9.2, MOTOR_TERMINAL.2, U11.2
- new net N$14: J5.1, R13.2
- new net N$15: J6.1, R11.2
- new net N$2: R12.2, SNUBBER.2
- net AGND: now also U5.4; no longer U$5.4
- net GND: now also C12.2, R11.1, R13.1, R14.1, U5.1, U5.2; no longer U$5.1, U$5.2
- net N$1: now also U5.3; no longer U$5.3
- net N$9: now also MOTOR_TERMINAL.1, SNUBBER.1, U11.1; no longer J3.1, R12.2, U$11.1
- net UNBIASED_VOLTAGE: now also U11.3; no longer U$11.3
- net VDD: now also C5.1, C6.1, D1.C, U11.5; no longer U$11.5
- net VDDA: now also U5.5; no longer C1.1, C2.1, U$5.5
- net VNEG: now also U11.4; no longer U$11.4
- net VPOS: now also C1.1, C2.1, J3.1, J3.2, J3.3; no longer C5.1, C6.1, D1.C
Routing:
- net VPOS: track 0.00 -> 43.8 mm
- net GND: track 0.00 -> 39.3 mm
- net N$4: track 0.00 -> 34.2 mm
- net 5V: track 0.00 -> 29.2 mm
- net UNBIASED_VOLTAGE: track 0.00 -> 27.9 mm
- net VNEG: track 0.00 -> 25.5 mm
- net N$6: track 0.00 -> 25.1 mm
- net BIASED_VOLTAGE: track 0.00 -> 16.6 mm
- net N$1: track 0.00 -> 16.3 mm
- net DAC_SCL: track 0.00 -> 15.1 mm
- net VCC-ISO: track 0.00 -> 14.4 mm
- net N$7: track 0.00 -> 10.2 mm
- net DAC_SDA: track 0.00 -> 9.85 mm
- net GND-ISO: track 0.00 -> 9.51 mm
- net N$3: track 0.00 -> 9.50 mm
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Other:
- board size 160 x 100 mm -> 79.8 x 100 mm
