File: Electronic/pcb/atlas_haptic_pcb/atlas_haptic_pcb/schematics.sch (EAGLE design)
At the start: 35 parts, among them U1 ISO1541, U3 MCP4725, U4 LM833N

Commit message: Figure of the circuit is updated. Mechanical part is revised.
Parts:
- removed U$11, U$5: OPA549, OPA:OPA549
- added C13: 1n, SparkFun-Capacitors:1.0UF-1206-50V-10%
- added D3, D4: (no value), adafruit:DIODEDO-1N4148
- added D5: (no value), adafruit:SCHOTTKY-DIODEAG
- added J5, J6, J7, J9, SNUBBER: Jumper, SparkFun-Connectors:CONN_02PTH3
- added MOTOR_TERMINAL, MOTOR_TERMINAL1: (no value), SparkFun-Connectors:CONN_025MM
- added R13: 0R1, SparkFun-Resistors:RESISTOR1206
- added R14, R23: 1R0, SparkFun-Resistors:RESISTOR1206
- added R15, R16, R17, R18, R19: 1k, SparkFun-Resistors:RESISTOR1206
- added R21: 10, SparkFun-Resistors:RESISTOR1206
- added U11, U5, U7: OPA549, OPA:OPA549
- added U6: LM833N, LM833N:LM833N
- C12: value 0.01uF -> 1n
- J3: device SparkFun-Connectors:CONN_025MM -> SparkFun-Connectors:CONN_03LONGPADS
- R11: value 0R1 -> 0R01
Connections:
- removed net N$8: J3.2, R11.2, U$11.-IN
- new net 1.55V: D3.A, R15.1, R16.1
- new net N$11: J7.1, J9.1, R14.2
- new net N$12: J5.2, J6.2, J7.2, J9.2, MOTOR_TERMINAL.2, U11.-IN
- new net N$13: R18.1, U6.-INA, U6.OUT_A
- new net N$14: J5.1, R13.2
- new net N$15: J6.1, R11.2
- new net N$16: C13.1, R21.1
- new net N$17: D3.C, D4.A
- new net N$18: D4.C, D5.A
- new net N$19: R16.2, R17.1, U6.-INB
- new net N$2: R12.2, SNUBBER.2
- new net N$20: MOTOR_TERMINAL1.1, R21.2, U7.OUT
- new net N$22: R18.2, R19.1, U6.+INB
- new net N$23: MOTOR_TERMINAL1.2, R23.2, U7.-IN
- net 3.3V: now also D5.C, R19.2; no longer C12.2, R11.1
- net AGND: now also U5.V-; no longer U$5.V-
- net BIASED_VOLTAGE: now also U6.+INA
- net GND: now also C12.2, C13.2, R11.1, R13.1, R14.1, R23.1, U5.-IN, U5.OUT; no longer U$5.-IN, U$5.OUT
- net N$1: now also U5.+IN; no longer U$5.+IN
- net N$9: now also MOTOR_TERMINAL.1, SNUBBER.1, U11.OUT; no longer J3.1, R12.2, U$11.OUT
- net UNBIASED_VOLTAGE: now also R17.2, U11.+IN, U6.OUT_B, U7.+IN; no longer U$11.+IN
- net VDD: now also C5.1, C6.1, D1.C, R15.2, U11.V+, U6.+VCC, U7.V+; no longer U$11.V+
- net VDDA: now also U5.V+; no longer C1.1, C2.1, U$5.V+
- net VNEG: now also U11.V-, U6.-VEE, U7.V-; no longer U$11.V-
- net VPOS: now also C1.1, C2.1, J3.1, J3.2, J3.3; no longer C5.1, C6.1, D1.C
Other:
- note added: "Analog Buffer"
- note added: "Current Sensing"
- note added: "Snubber Circuit"
- note added: "Voltage Subtractor"
- moved on the sheet: C1, C10, C11, C12, C2, C3, C4, C5, C6, C7, C8, C9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
